Commit message: Separated ground_plane and sun from track xacros

File: simulation/models/tracks/acceleration.xacro (robot description, xacro)
@@ -13,62 +13,12 @@
         name="gz::sim::systems::UserCommands">
       </plugin>
-	  <xacro:include filename="$(find simulation)/models/tracks/physics.urdf.xacro"/>
+	  <xacro:include filename="$(find simulation)/models/world/physics.xacro"/>
     <xacro:physics_tags/>
-    <!-- <include>
-      <uri>model://sun</uri>
-    </include> -->
-    <light type="directional" name="sun">
-      <cast_shadows>true</cast_shadows>
-      <pose>0 0 10 0 0 0</pose>
-      <diffuse>1 1 1 1</diffuse>
-      <specular>0.5 0.5 0.5 1</specular>
-      <attenuation>
-        <range>1000</range>
-        <constant>0.9</constant>
-        <linear>0.01</linear>
-        <quadratic>0.001</quadratic>
-      </attenuation>
-      <direction>-0.5 0.1 -0.9</direction>
-    </light>
-    <!-- <include>
-      <uri>model://ground_plane</uri>
-    </include> -->
-    <model name="ground_plane">
-      <static>true</static>
-      <link name="link">
-        <collision name="collision">
-          <geometry>
-            <plane>
-              <normal>0 0 1</normal>
-              <size>120 120</size>
-            </plane>
-          </geometry>
-          <surface>
-            <friction>
-              <ode>
-                <mu>50</mu>
-              </ode>
-              <bullet>
-                <friction>1</friction>
-                <rolling_friction>0.1</rolling_friction>
-              </bullet>
-            </friction>
-          </surface>
-        </collision>
-        <visual name="visual">
-          <geometry>
-            <plane>
-              <normal>0 0 1</normal>
-              <size>120 120</size>
-            </plane>
-          </geometry>
-          <material>
-            <ambient>0.8 0.8 0.8 1</ambient>
-            <diffuse>0.8 0.8 0.8 1</diffuse>
-            <specular>0.8 0.8 0.8 1</specular>
-          </material>
-        </visual>
-      </link>
-    </model>
+    <include>
+      <uri>model://simulation/models/world/sun</uri>
+    </include>
+    <include>
+      <uri>model://simulation/models/world/ground_plane</uri>
+    </include>
     <xacro:include filename="$(find simulation)/models/cones/cone.sdf.xacro"/>
     <model name='cones'>

File: simulation/models/tracks/skidpad.xacro (robot description, xacro)
@@ -13,62 +13,12 @@
         name="gz::sim::systems::UserCommands">
       </plugin>
-    <xacro:include filename="$(find simulation)/models/tracks/physics.urdf.xacro"/>
+    <xacro:include filename="$(find simulation)/models/world/physics.xacro"/>
     <xacro:physics_tags/>
-    <!-- <include>
-      <uri>model://sun</uri>
-    </include> -->
-    <light type="directional" name="sun">
-      <cast_shadows>true</cast_shadows>
-      <pose>0 0 10 0 0 0</pose>
-      <diffuse>1 1 1 1</diffuse>
-      <specular>0.5 0.5 0.5 1</specular>
-      <attenuation>
-        <range>1000</range>
-        <constant>0.9</constant>
-        <linear>0.01</linear>
-        <quadratic>0.001</quadratic>
-      </attenuation>
-      <direction>-0.5 0.1 -0.9</direction>
-    </light>
-    <!-- <include>
-      <uri>model://ground_plane</uri>
-    </include> -->
-    <model name="ground_plane">
-      <static>true</static>
-      <link name="link">
-        <collision name="collision">
-          <geometry>
-            <plane>
-              <normal>0 0 1</normal>
-              <size>100 100</size>
-            </plane>
-          </geometry>
-          <surface>
-            <friction>
-              <ode>
-                <mu>50</mu>
-              </ode>
-              <bullet>
-                <friction>1</friction>
-                <rolling_friction>0.1</rolling_friction>
-              </bullet>
-            </friction>
-          </surface>
-        </collision>
-        <visual name="visual">
-          <geometry>
-            <plane>
-              <normal>0 0 1</normal>
-              <size>100 100</size>
-            </plane>
-          </geometry>
-          <material>
-            <ambient>0.8 0.8 0.8 1</ambient>
-            <diffuse>0.8 0.8 0.8 1</diffuse>
-            <specular>0.8 0.8 0.8 1</specular>
-          </material>
-        </visual>
-      </link>
-    </model>
+    <include>
+      <uri>model://simulation/models/world/sun</uri>
+    </include>
+    <include>
+      <uri>model://simulation/models/world/ground_plane</uri>
+    </include>
     <xacro:include filename="$(find simulation)/models/cones/cone.sdf.xacro"/>
     <model name="cones">

File: simulation/models/tracks/track_small.xacro (robot description, xacro)
@@ -2,62 +2,12 @@
 <sdf version='1.7' xmlns:xacro="http://www.ros.org/wiki/xacro">
   <world name='map'>
-    <xacro:include filename="$(find simulation)/models/tracks/physics.urdf.xacro"/>
+    <xacro:include filename="$(find simulation)/models/world/physics.xacro"/>
     <xacro:physics_tags/>
-    <!-- <include>
-      <uri>model://sun</uri>
-    </include> -->
-    <light type="directional" name="sun">
-      <cast_shadows>true</cast_shadows>
-      <pose>0 0 10 0 0 0</pose>
-      <diffuse>1 1 1 1</diffuse>
-      <specular>0.5 0.5 0.5 1</specular>
-      <attenuation>
-        <range>1000</range>
-        <constant>0.9</constant>
-        <linear>0.01</linear>
-        <quadratic>0.001</quadratic>
-      </attenuation>
-      <direction>-0.5 0.1 -0.9</direction>
-    </light>
-    <!-- <include>
-      <uri>model://ground_plane</uri>
-    </include> -->
-    <model name="ground_plane">
-      <static>true</static>
-      <link name="link">
-        <collision name="collision">
-          <geometry>
-            <plane>
-              <normal>0 0 1</normal>
-              <size>100 100</size>
-            </plane>
-          </geometry>
-          <surface>
-            <friction>
-              <ode>
-                <mu>50</mu>
-              </ode>
-              <bullet>
-                <friction>1</friction>
-                <rolling_friction>0.1</rolling_friction>
-              </bullet>
-            </friction>
-          </surface>
-        </collision>
-        <visual name="visual">
-          <geometry>
-            <plane>
-              <normal>0 0 1</normal>
-              <size>100 100</size>
-            </plane>
-          </geometry>
-          <material>
-            <ambient>0.8 0.8 0.8 1</ambient>
-            <diffuse>0.8 0.8 0.8 1</diffuse>
-            <specular>0.8 0.8 0.8 1</specular>
-          </material>
-        </visual>
-      </link>
-    </model>
+    <include>
+      <uri>model://simulation/models/world/sun</uri>
+    </include>
+    <include>
+      <uri>model://simulation/models/world/ground_plane</uri>
+    </include>
     <xacro:include filename="$(find simulation)/models/cones/cone.sdf.xacro"/>
     <model name="cones">

File: simulation/models/world/physics.xacro (robot description, xacro)
@@ -1,4 +1,4 @@
 <?xml version="1.0" ?>
-<robot xmlns:xacro="http://www.ros.org/wiki/xacro">
+<sdf version='1.7' xmlns:xacro="http://www.ros.org/wiki/xacro">
     <xacro:macro name="physics_tags" params="">
         <gravity>0 0 -9.8</gravity>
@@ -24,3 +24,3 @@
         </spherical_coordinates>
     </xacro:macro>
-</robot>
+</sdf>
